File: Hardware/Circuit and PCB/WattMeter.kicad_pcb (KiCad board)
At the start: 2 copper layers, 185 x 126.1 mm, 80 parts, among them IC1 ATM90E32AS-AU-R, IC2 LM2621MMX_NOPB, J1 LCD Pins, J10 I2 Use/GND, J11 Input, J12 V3 Use/GND, J13 I1, J14 Series/Para, J15 Series/Para, J16 V2 Use/GND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

Commit message: Add some plots
Parts:
- removed REF**: 1591XXF Enclosure 4 point, Mounting Footprints:1591XXF Enclosure 4 point
- added N1: Housing, Mounting Footprints:1591XXF Enclosure 4 point, F.Cu at (60.7, 50.4)
- R5: value 500Ω -> 499Ω
