File: Hardware/Circuit and PCB/WattMeter.kicad_sch (KiCad schematic)
At the start: 78 parts, among them IC1 ATM90E32AS-AU-R, IC2 LM2621MMX_NOPB, J1 LCD Pins, J10 I2 Use/GND, J11 Input, J12 V3 Use/GND, J13 I1, J14 Series/Para, J15 Series/Para, J16 V2 Use/GND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

Commit message: Add some plots
Parts:
- added N1: Housing, Mounting Footprints:1591XXF Enclosure 4 point, symbol Mechanical:Housing
- C4: Mouser Link (none) -> https://www.mouser.com/ProductDetail/Vishay-BC-Components/K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; Mouser# (none) -> 594-K104K15X7RF53L2; Price/unit (none) -> 0.106
- D1: Mouser# 511-1N5822 -> 511-1N5822
- D4: Mouser Link (none) -> https://www.mouser.com/ProductDetail/Vishay-Semiconductors/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; Mouser# (none) -> 78-1N4734A; Price/unit (none) -> 0.052
- D5, D6: Mouser Link (none) -> https://www.mouser.com/ProductDetail/LITEON/LTL-4213?qs=o%2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; Mouser# (none) -> 859-LTL-4213; Price/unit (none) -> 0.088
- IC2: Price/unit (none) -> 1.77
- J1: Mouse Link (none) -> https://www.mouser.com/ProductDetail/Chip-Quik/HDR100IMP40M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; Mouser# (none) -> 910-HDR100IMP40MGVTH; Price/unit (none) -> 0.058
- J10, J12, J14, J15, J16, J5, J9: Mouser# (none) -> 910-HDR100IMP40MGVTH; Price/unit (none) -> 0.058
- J13, J17, J18, J19: Mouser# (none) -> 910-HDR100IMP40MGVTH; Price/unit (none) -> 0.029
- J2: Mouse Link (none) -> https://www.mouser.com/ProductDetail/Chip-Quik/HDR100IMP40M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; Mouser# (none) -> 910-HDR100IMP40MGVTH; Price/unit (none) -> 0.0145
- J4: Mouse Link (none) -> https://www.mouser.com/ProductDetail/Chip-Quik/HDR100IMP40M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; Mouser# (none) -> 910-HDR100IMP40MGVTH; Price/unit (none) -> 0.145
- J6, J7, J8: now left out of the parts list
- L1: Price/unit (none) -> 1.65
- R1, R2, R4, R7: Mouser# (none) -> 603-MFR-25FTE52-10K; Price/unit (none) -> 0.028
- R10, R11: Mouser# (none) -> MFR-25FBF52-100R; Price/unit (none) -> 0.029
- R12, R13: Mouser# (none) -> 603-MFR-25FBF52-5K1; Price/unit (none) -> 0.029
- R14, R18: Mouser# (none) -> 603-MFR-25FBF52-1K; Price/unit (none) -> 0.026
- R19: Mouser# (none) -> 603-MFR-25FBF52-24K; Price/unit (none) -> 0.029
- R3: Mouser# (none) -> 603-MFR-25FBF52-200K; Price/unit (none) -> 0.029
- R5: value 500Ω -> 499Ω; Mouser# (none) -> 603-MFR-25FBF52-499R; Price/unit (none) -> 0.027
- R6: Mouser# (none) -> 603-MFR-25FBF52-12K; Price/unit (none) -> 0.029
- R8: Price/unit (none) -> 1.46
- R9: Mouser# (none) -> 603-MFR-25FBF52-30R; Price/unit (none) -> 0.029
- RV2: Mouser Link (none) -> https://www.mouser.com/ProductDetail/Bourns/PV36W204C01B00?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; Mouser# (none) -> 81-PV36W204C01B00; Price/unit (none) -> 1.21
- U1: Mouser# (none) -> 356-ESP32C6DKC1N8; Price/unit 12.48 -> 8.76
Other:
- title: (none) -> WattMeter
- moved on the sheet: C13, J11, J6, J7, J8, P1, P2
